File: hardware/kicad-proj/remote-monitor.sch (KiCad schematic (older format))
At the start: 13 parts

Commit message: prototype main board complete
Parts:
- removed D? (x2): D_ALT, symbol Device:D_ALT
- removed J?: Screw_Terminal_01x04, symbol Connector:Screw_Terminal_01x04
- removed J?: Screw_Terminal_01x02, symbol Connector:Screw_Terminal_01x02
- removed U? (x2): DC/DC Converter, Converter_DCDC:Converter_DCDC_RECOM_R-78B-2.0_THT, symbol Regulator_Switching:R-78B5.0-2.0
- added C3, C4: 100nf, Capacitor_SMD:C_1206_3216Metric, symbol Device:C
- added C5, C6, C9: 1uf, Capacitor_SMD:C_1206_3216Metric, symbol Device:C
- added C7, C8: C, Capacitor_SMD:C_1206_3216Metric, symbol Device:C
- added D2, D3, D4: BAT54S, Package_TO_SOT_SMD:SOT-23, symbol Diode:BAT54S
- added F1, F2: 1A, Fuse:Fuse_1812_4532Metric, symbol Device:Polyfuse
- added J1: Screw_Terminal_01x10, remote-monitor:Screw_Terminal_1x10, symbol Connector:Screw_Terminal_01x10
- added R2: 100R, Resistor_SMD:R_1206_3216Metric, symbol Device:R
- added R4: 10k, Resistor_SMD:R_1206_3216Metric, symbol Device:R
- added R5, R6: 1K, Resistor_SMD:R_1206_3216Metric, symbol Device:R
- added U1, U2: OKI-78SR-5, Converter_DCDC:Converter_DCDC_muRata_OKI-78SR_Vertical, symbol 1.remote-monitor:OKI-78SR-5
- A1: renamed from A?; footprint (none) -> remote-monitor:Arduino_MKR_1010
- C1: renamed from C?; footprint (none) -> Capacitor_SMD:CP_Elec_5x4.5
- C2: renamed from C?; footprint (none) -> Capacitor_SMD:C_1206_3216Metric
- D1: renamed from D?; value D_ALT -> SMA; footprint (none) -> Diode_SMD:D_SMA; symbol Device:D_ALT -> Device:D_Schottky
- J2: renamed from J?; footprint (none) -> remote-monitor:USB_A_Molex_105057_Vertical
- R1: renamed from R?; value 5K -> 10k; footprint (none) -> Resistor_SMD:R_1206_3216Metric
- R3: renamed from R?; value 1K -> 2k; footprint (none) -> Resistor_SMD:R_1206_3216Metric
Connections:
- net Mains_Sensor_Out is gone; now on net Mains_Sensor: A1.3 (A1)
- net +3V3: now also A1.26 (3V3), D2.2, D3.2, D4.2
- net +5V: now also C8.1, U2.3 (OUT)
- net Battery_Volts: now also D2.3
- net GND: now also J2.4 (GND), J2.5 (Shield), C3.2, C4.2, C5.2, C6.2, C7.2, C8.2, D2.1, D3.1, D4.1, J1.4 (Pin_4), J1.5 (Pin_5), J1.6 (Pin_6), R4.1, R6.2, U1.2 (GND), U2.2 (GND)
- net at C1.1, D1.1 (K): now also C4.1, C5.1, C6.1, U1.1 (IN), U2.1 (IN); no longer R1.2
- net at D1.2 (A): now also F1.1
- net Mains_Sensor: now reaches A1.15 (D6)
- net Mains_Sensor: now also A1.16 (D7), C3.1, D3.3, R2.1, R4.2
- net at A1.2 (DAC0/A0): now also C9.2, D4.3
- net at J2.1 (VBUS): now also F2.1
- net at J2.2 (D-): now also J2.3 (D+)
- new net: F1.2, J1.1 (Pin_1), J1.2 (Pin_2), J1.3 (Pin_3), R1.2
- new net: C7.1, F2.2, U1.3 (OUT)
- new net: C9.1, R5.1
- new net: J1.8 (Pin_8), R2.2
- new net Radio_VOX: J1.10 (Pin_10), R5.2, R6.1
- no-connect marks 0 -> 22
Other:
- note added: "0"
- note added: "29/08/20"
- note added: "Erik Stefan\n2020\nCC BY-NC 3.0 AU"
- note added: "Remote Monitor Main Board"
- moved on the sheet: A1, C1, C2, J2, R1, R3

Commit message: updated hardware designs
Parts:
- added C10, C11: 4.7uf, Capacitor_SMD:C_1206_3216Metric, symbol Device:C
- added C12: 470uf, Capacitor_SMD:CP_Elec_8x10.5, symbol Device:CP
- added C13: 100nf, Capacitor_SMD:C_1206_3216Metric, symbol Device:C
- added L1: 1mH, Inductor_SMD:L_6.3x6.3_H3, symbol Device:L
- added U3: NCP51460, Package_TO_SOT_SMD:SOT-23, symbol 1.remote-monitor:NCP51460
- C1: value 10uF -> 10uf
- C3: value 100nf -> 1nf
- C7, C8: value C -> 1uf
- F1, F2: value 1A -> 0.5A
- J1: value Screw_Terminal_01x10 -> Screw Terminal
- R4: value 10k -> 100k
- R6: value 1K -> 100k
Connections:
- net +3V3: no longer D3.2
- net +5V: now also C12.1, C13.1, L1.1, U3.1 (Vin); no longer C8.1, U2.3 (OUT)
- net GND: now also C10.2, C12.2, C13.2, U3.3 (GND); no longer R6.2
- net Mains_Sensor: now also R6.1; no longer A1.15 (D6), A1.16 (D7)
- net AREF: now reaches A1.1 (AREF)
- net AREF: now also D3.2, R6.2, U3.2 (Vout)
- net at J1.8 (Pin_8): now also C11.1; no longer R2.2
- net Radio_GND: now reaches J1.9 (Pin_9)
- net Radio_GND: now also C10.1
- net Radio_VOX renamed Radio_Sig
- net Radio_Sig: no longer R6.1
- new net: C8.1, L1.2, U2.3 (OUT)
- new net: C11.2, R2.2
Other:
- note added: "+12V"
- note added: "0.1"
- note added: "18/10/20"
- note added: "AC\nAmplifier"
- note added: "GND"
- note added: "Repeater Monitor Main Board"
- note added: "To Radio"
- note removed: "0"
- note removed: "29/08/20"
- note removed: "Remote Monitor Main Board"
- moved on the sheet: C1, C2, C3, C4, C5, C6, C7, C8, D1, D2, D3, F1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
